File: hw/fjarr.kicad_sch (KiCad schematic)
At the start: 13 parts, among them Q1 2N2219, U1 TSOP48xx, U3 ESP32-C3-DevKitM-1

Commit message: Design update for v0.1 build
Parts:
- removed Q1: 2N2219, Package_TO_SOT_THT:TO-39-3, symbol Transistor_BJT:2N2219
- removed U3: ESP32-C3-DevKitM-1, RF_Module:ESP32-C3-DevKitM-1, symbol RF_Module:ESP32-C3-DevKitM-1
- added C3: 22u, Capacitor_SMD:C_0805_2012Metric, symbol Device:C
- added C4: 10u, Capacitor_SMD:C_0805_2012Metric, symbol Device:C
- added C5: 1n, Capacitor_SMD:C_0805_2012Metric, symbol Device:C
- added C6: 100n, Capacitor_SMD:C_0402_1005Metric, symbol Device:C
- added D4: SMAJ5.0A, Diode_SMD:D_SMA, symbol Diode:SMAJ5.0A
- added D5: LED, LED_SMD:LED_0805_2012Metric, symbol Device:LED
- added H1, H2, H3: MountingHole, MountingHole:MountingHole_2.2mm_M2, symbol Mechanical:MountingHole
- added Q2: AO3400A, Package_TO_SOT_SMD:SOT-23, symbol Transistor_FET:AO3400A
- added R10, R12, R13, R7: 10k, Resistor_SMD:R_0402_1005Metric, symbol Device:R
- added R11: 220, Resistor_SMD:R_0402_1005Metric, symbol Device:R
- added R6: 33, Resistor_SMD:R_0402_1005Metric, symbol Device:R
- added R8, R9: 5.1k, Resistor_SMD:R_0402_1005Metric, symbol Device:R
- added SW1: SW_Push, PCM_JLCPCB:SW_TS-1088-AR02016, symbol Switch:SW_Push
- added TP1, TP2, TP3, TP4, TP5, TP6, TP7: TestPoint, TestPoint:TestPoint_Pad_D1.0mm, symbol Connector:TestPoint
- added U2: AMS1117-3.3, Package_TO_SOT_SMD:SOT-223-3_TabPin2, symbol Regulator_Linear:AMS1117-3.3
- added U3: USBLC6-2P6, Package_TO_SOT_SMD:SOT-666, symbol Power_Protection:USBLC6-2P6
- added U4: (no value), EasyEDA_Lib:TYPE-C-SMD_HX-TYPE-C-16PIN, symbol EasyEDA_Lib:HX TYPE-C 16PIN
- added U5: ESP32-C3-WROOM-02, PCM_Espressif:ESP32-C3-WROOM-02, symbol PCM_Espressif:ESP32-C3-WROOM-02
- C1: footprint (none) -> Capacitor_SMD:C_0805_2012Metric
- C2: value 10u -> 100n; footprint (none) -> Capacitor_SMD:C_0402_1005Metric
- D1, D2, D3: footprint LED_THT:LED_D3.0mm_IRBlack -> LED_THT:LED_D5.0mm_IRBlack; now left out of the parts list
- R1, R2: footprint (none) -> Resistor_SMD:R_0402_1005Metric
- R3: value 47 -> 10k; footprint (none) -> Resistor_SMD:R_0402_1005Metric
- R4, R5: value 47 -> 33; footprint (none) -> Resistor_SMD:R_0402_1005Metric
- U1: value TSOP48xx -> TSOP4838
Connections:
- net +3.3V: now also C3.1, R10.2, R12.2, R13.2, R7.2, TP6.1, U2.2 (VO), U5.1 (3V3)
- net +5V: now also C4.1, D4.1 (A1), R6.2, TP5.1, U2.3 (VI), U3.5 (VBUS), U4.A9B4 (VBUS), U4.B9A4 (VBUS); no longer R3.2
- net GND: now also R3.1, C3.2, C4.2, C5.2, C6.2, D4.2 (A2), D5.1 (K), Q2.2 (S), R8.2, R9.2, SW1.1, TP7.1, U2.1 (GND), U3.2 (GND), U4.A12B1 (GND), U4.B12A1 (GND), U5.19 (GND), U5.9 (GND)
- net IR_RX: now also TP1.1, U5.18 (GPIO0/ADC1_CH0/XTAL_32K_P)
- net IR_TX: now also TP2.1, U5.17 (GPIO1/ADC1_CH1/XTAL_32K_N)
- net at R5.1: now also D2.2 (A); no longer D3.2 (A)
- net at D1.1 (K), D2.1 (K), D3.1 (K): now also Q2.3 (D)
- net at D1.2 (A): now also R4.1; no longer R3.1
- net at R2.1: now also R3.2, Q2.1 (G)
- new net: R13.1, U5.16 (GPIO2/ADC1_CH2)
- new net: R7.1, U5.2 (EN/CHIP_PU)
- new net: R12.1, U5.7 (GPIO8)
- new net: C5.1, U4.17 (EH), U4.18 (EH), U4.19 (EH), U4.20 (EH)
- new net: D3.2 (A), R6.1
- new net: D5.2 (A), R11.2
- new net BOOT: C6.1, R10.1, SW1.2, U5.8 (GPIO9)
- new net CC1: R8.1, U4.A5 (CC1)
- new net CC2: R9.1, U4.B5 (CC2)
- new net CD+: U3.3 (I/O2), U4.A6 (D+), U4.B6 (D+)
- new net CD-: U3.1 (I/O1), U4.A7 (D-), U4.B7 (D-)
- new net D+: TP3.1, U3.4 (I/O2), U5.13 (GPIO18/USB_D-)
- new net D-: TP4.1, U3.6 (I/O1), U5.14 (GPIO19/USB_D+)
- new net LED: R11.1, U5.6 (GPIO7)
- no-connect marks 0 -> 2
Other:
- note added: "IR Receiver"
- note added: "Power"
- note added: "Usb"
- note removed: "IR Reciver"
- moved on the sheet: C1, R1, U1
